File: RC_v2_ESP32/RC_v2_ESP32.kicad_pcb (KiCad board)
At the start: 2 copper layers, 13 parts, among them SW3 SW_DIP_x01, SW4 SW_DIP_x01, SW5 SW_DIP_x01, SW6 SW_DIP_x01

Commit message: bearbeitung
Parts:
- removed U2: ~, Amjad_lib:MPU_6050_bord
- moved RV2 66.3 mm to (119.0, 54.2), turned to -90 degrees
- moved RV3 58.7 mm to (118.4, 74.2)
- moved RV1 47.5 mm to (118.5, 93.5)
Changed lines of the file:
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@@
 	)
 	(setup
+		(stackup
+			(layer "F.SilkS"
+				(type "Top Silk Screen")
+			)
+			(layer "F.Paste"
+				(type "Top Solder Paste")
+			)
+			(layer "F.Mask"
+				(type "Top Solder Mask")
+				(thickness 0.01)
+			)
+			(layer "F.Cu"
+				(type "copper")
+				(thickness 0.035)
+			)
+			(layer "dielectric 1"
+				(type "core")
+				(thickness 1.51)
+				(material "FR4")
+				(epsilon_r 4.5)
+				(loss_tangent 0.02)
+			)
+			(layer "B.Cu"
+				(type "copper")
+				(thickness 0.035)
+			)
+			(layer "B.Mask"
+				(type "Bottom Solder Mask")
+				(thickness 0.01)
+			)
+			(layer "B.Paste"
+				(type "Bottom Solder Paste")
+			)
+			(layer "B.SilkS"
+				(type "Bottom Silk Screen")
+			)
+			(copper_finish "None")
+			(dielectric_constraints no)
+		)
 		(pad_to_mask_clearance 0)
 		(allow_soldermask_bridges_in_footprints no)
@@
 	(net 49 "unconnected-(U1-G17-Pad30)")
 	(net 50 "unconnected-(U1-G18-Pad28)")
-	(net 51 "unconnected-(U2-XCL-Pad6)")
-	(net 52 "unconnected-(U2-VCC-Pad1)")
-	(net 53 "unconnected-(U2-SCL-Pad3)")
-	(net 54 "unconnected-(U2-ADO-Pad7)")
-	(net 55 "unconnected-(U2-SDA-Pad4)")
-	(net 56 "unconnected-(U2-INT-Pad8)")
-	(net 57 "unconnected-(U2-GND-Pad2)")
-	(net 58 "unconnected-(U2-XDA-Pad5)")
 	(footprint "Library_Amjad:ESP_32_socket"
 		(layer "F.Cu")
@@
 		)
 	)
-	(footprint "Amjad_lib:MPU_6050_bord"
-		(layer "F.Cu")
-		(at 122.4 62.1)
-		(property "Reference" "U2"
-			(at -6.4 -7.884 0)
-			(unlocked yes)
-			(layer "F.SilkS")
-			(effects
-				(font
-					(size 1 1)
-					(thickness 0.1)
-				)
-			)
-		)
-		(property "Value" "~"
-			(at -6.4 -5.852 0)
-			(unlocked yes)
-			(layer "F.Fab")
-			(effects
-				(font
-					(size 1 1)
-					(thickness 0.15)
-				)
-			)
-		)
-		(property "Datasheet" ""
-			(at -6.4 3.8 0)
-			(unlocked yes)
-			(layer "F.Fab")
-			(hide yes)
-			(effects
-				(font
-					(size 1 1)
-					(thickness 0.15)
-				)
-			)
-		)
-		(property "Description" ""
-			(at -6.4 3.8 0)
-			(unlocked yes)
-			(layer "F.Fab")
-			(hide yes)
-			(effects
-				(font
-					(size 1 1)
-					(thickness 0.15)
-				)
-			)
-		)
-		(sheetname "/")
-		(sheetfile "RC_v2_ESP32.kicad_sch")
-		(attr smd)
-		(fp_rect
-			(start -13.9 -1.1)
-			(end 1.1 18.9)
-			(stroke
-				(width 0.1)
-				(type default)
-			)
-			(fill no)
-			(layer "F.SilkS")
-		)
-		(fp_text user "${REFERENCE}"
-			(at -6.4 -4.328 0)
-			(unlocked yes)
-			(layer "F.Fab")
-			(effects
-				(font
-					(size 1 1)
-					(thickness 0.15)
-				)
-			)
-		)
-		(pad "1" thru_hole oval
-			(at 0 0)
-			(size 1.7 1.7)
-			(drill 1)
-			(layers "*.Cu" "*.Mask")
-			(remove_unused_layers no)
-			(net 52 "unconnected-(U2-VCC-Pad1)")
-			(pinfunction "VCC")
-			(pintype "input")
-		)
-		(pad "2" thru_hole oval
-			(at 0 2.54)
-			(size 1.7 1.7)
-			(drill 1)
-			(layers "*.Cu" "*.Mask")
-			(remove_unused_layers no)
-			(net 57 "unconnected-(U2-GND-Pad2)")
-			(pinfunction "GND")
-			(pintype "input")
-		)
-		(pad "3" thru_hole oval
-			(at 0 5.08)
-			(size 1.7 1.7)
-			(drill 1)
-			(layers "*.Cu" "*.Mask")
-			(remove_unused_layers no)
-			(net 53 "unconnected-(U2-SCL-Pad3)")
-			(pinfunction "SCL")
-			(pintype "input")
-		)
-		(pad "4" thru_hole oval
-			(at 0 7.62)
-			(size 1.7 1.7)
-			(drill 1)
-			(layers "*.Cu" "*.Mask")
-			(remove_unused_layers no)
-			(net 55 "unconnected-(U2-SDA-Pad4)")
-			(pinfunction "SDA")
-			(pintype "input")
-		)
-		(pad "5" thru_hole oval
-			(at 0 10.16)
-			(size 1.7 1.7)
-			(drill 1)
-			(layers "*.Cu" "*.Mask")
-			(remove_unused_layers no)
-			(net 58 "unconnected-(U2-XDA-Pad5)")
-			(pinfunction "XDA")
-			(pintype "input")
-		)
-		(pad "6" thru_hole oval
-			(at 0 12.7)
-			(size 1.7 1.7)
-			(drill 1)
-			(layers "*.Cu" "*.Mask")
-			(remove_unused_layers no)
-			(net 51 "unconnected-(U2-XCL-Pad6)")
-			(pinfunction "XCL")
-			(pintype "input")
-		)
-		(pad "7" thru_hole oval
-			(at 0 15.24)
-			(size 1.7 1.7)
-			(drill 1)
-			(layers "*.Cu" "*.Mask")
-			(remove_unused_layers no)
-			(net 54 "unconnected-(U2-ADO-Pad7)")
-			(pinfunction "ADO")
-			(pintype "input")
-		)
-		(pad "8" thru_hole oval
-			(at 0 17.78)
-			(size 1.7 1.7)
-			(drill 1)
-			(layers "*.Cu" "*.Mask")
-			(remove_unused_layers no)
-			(net 56 "unconnected-(U2-INT-Pad8)")
-			(pinfunction "INT")
-			(pintype "input")
-		)
-		(embedded_fonts no)
-	)
 	(footprint "Resistor_SMD:R_1206_3216Metric"
 		(layer "F.Cu")
@@
 	(footprint "Potentiometer_THT:Potentiometer_Alps_RK09K_Single_Vertical"
 		(layer "F.Cu")
-		(at 53.4575 44.41)
+		(at 119 54.25 -90)
 		(descr "113004U 1130A6S 11300DR 1130A8G 1130081 1130A5R 1130AP5 1130AST  D1130C3W D1130C1B D1130C3C D1130C2P Potentiometer, vertical, Alps RK09K Single, https://tech.alpsalpine.com/prod/e/pdf/potentiometer/rotarypotentiometers/rk09k/rk09k.pdf")
 		(tags "Potentiometer vertical Alps RK09K RK09D Single Snapin")
 		(property "Reference" "RV2"
-			(at 6.05 -5.15 0)
+			(at 6.05 -5.15 90)
 			(layer "F.SilkS")
 			(effects
@@
 		)
 		(property "Value" "R_Potentiometer_Small"
-			(at 6.05 10.15 0)
+			(at 6.05 10.15 90)
 			(layer "F.Fab")
 			(effects
@@
 		)
 		(property "Datasheet" ""
-			(at 0 0 0)
+			(at 0 0 270)
 			(unlocked yes)
 			(layer "F.Fab")
@@
 		)
 		(property "Description" "Potentiometer"
-			(at 0 0 0)
+			(at 0 0 270)
 			(unlocked yes)
 			(layer "F.Fab")
@@
 		(attr through_hole)
 		(fp_line
-			(start 0.88 -2.521)
-			(end 0.88 -1.2)
+			(start 0.88 7.52)
+			(end 4.817 7.52)
 			(stroke
 				(width 0.12)
@@
 		)
 		(fp_line
-			(start 0.88 -2.521)
-			(end 4.817 -2.521)
+			(start 9.184 7.52)
+			(end 13.12 7.52)
 			(stroke
 				(width 0.12)
@@
 		)
 		(fp_line
-			(start 0.88 1.25)
-			(end 0.88 1.63)
+			(start 0.88 5.87)
+			(end 0.88 7.52)
 			(stroke
 				(width 0.12)
@@
 		)
 		(fp_line
-			(start 0.88 5.87)
-			(end 0.88 7.52)
+			(start 0.88 1.25)
+			(end 0.88 1.63)
 			(stroke
 				(width 0.12)
@@
 		)
 		(fp_line
-			(start 0.88 7.52)
-			(end 4.817 7.52)
+			(start 0.88 -2.521)
+			(end 0.88 -1.2)
 			(stroke
 				(width 0.12)
@@
 		)
 		(fp_line
-			(start 9.184 -2.521)
-			(end 13.12 -2.521)
+			(start 0.88 -2.521)
+			(end 4.817 -2.521)
 			(stroke
 				(width 0.12)
@@
 		)
 		(fp_line
-			(start 9.184 7.52)
-			(end 13.12 7.52)
+			(start 9.184 -2.521)
+			(end 13.12 -2.521)
 			(stroke
 				(width 0.12)
@@
 		)
 		(fp_line
-			(start -1.15 -4.15)
-			(end -1.15 9.15)
+			(start -1.15 9.15)
+			(end 13.25 9.15)
 			(stroke
 				(width 0.05)
@@
 		)
 		(fp_line
-			(start -1.15 9.15)
-			(end 13.25 9.15)
+			(start 13.25 9.15)
+			(end 13.25 -4.15)
 			(stroke
 				(width 0.05)
@@
 		)
 		(fp_line
-			(start 13.25 -4.15)
-			(end -1.15 -4.15)
+			(start -1.15 -4.15)
+			(end -1.15 9.15)
 			(stroke
 				(width 0.05)
@@
 		)
 		(fp_line
-			(start 13.25 9.15)
-			(end 13.25 -4.15)
+			(start 13.25 -4.15)
+			(end -1.15 -4.15)
 			(stroke
 				(width 0.05)
@@
 		)
 		(fp_line
-			(start 1 -2.4)
-			(end 1 7.4)
+			(start 1 7.4)
+			(end 13 7.4)
 			(stroke
 				(width 0.1)
@@
 		)
 		(fp_line
-			(start 1 7.4)
-			(end 13 7.4)
+			(start 13 7.4)
+			(end 13 -2.4)
 			(stroke
 				(width 0.1)
@@
 		)
 		(fp_line
-			(start 13 -2.4)
-			(end 1 -2.4)
+			(start 1 -2.4)
+			(end 1 7.4)
 			(stroke
 				(width 0.1)
@@
 		)
 		(fp_line
-			(start 13 7.4)
-			(end 13 -2.4)
+			(start 13 -2.4)
+			(end 1 -2.4)
 			(stroke
 				(width 0.1)
@@
 		)
 		(fp_text user "${REFERENCE}"
-			(at 2 2.5 90)
+			(at 2 2.5 0)
 			(layer "F.Fab")
 			(effects
@@
 		)
 		(pad "1" thru_hole rect
-			(at 0 0)
+			(at 0 0 270)
 			(size 1.8 1.8)
 			(drill 1)
@@
 		)
 		(pad "2" thru_hole circle
-			(at 0 2.5)
+			(at 0 2.5 270)
 			(size 1.8 1.8)
 			(drill 1)
@@
 		)
 		(pad "3" thru_hole circle
-			(at 0 5)
+			(at 0 5 270)
 			(size 1.8 1.8)
 			(drill 1)
@@
 		)
 		(pad "MP" thru_hole roundrect
-			(at 7 -1.9)
+			(at 7 -1.9 270)
 			(size 4 3)
 			(drill oval 2.1 1.8)
@@
 		)
 		(pad "MP" thru_hole roundrect
-			(at 7 6.9)
+			(at 7 6.9 270)
 			(size 4 3)
 			(drill oval 2.1 1.8)
@@
 	(footprint "Potentiometer_THT:Potentiometer_Alps_RK09K_Single_Vertical"
 		(layer "F.Cu")
-		(at 87.5 57.45 -90)
+		(at 118.5 93.45 -90)
 		(descr "113004U 1130A6S 11300DR 1130A8G 1130081 1130A5R 1130AP5 1130AST  D1130C3W D1130C1B D1130C3C D1130C2P Potentiometer, vertical, Alps RK09K Single, https://tech.alpsalpine.com/prod/e/pdf/potentiometer/rotarypotentiometers/rk09k/rk09k.pdf")
 		(tags "Potentiometer vertical Alps RK09K RK09D Single Snapin")
@@
 	(footprint "Potentiometer_THT:Potentiometer_Alps_RK09K_Single_Vertical"
 		(layer "F.Cu")
-		(at 61.6 59.5 -90)
+		(at 118.4 74.15 -90)
 		(descr "113004U 1130A6S 11300DR 1130A8G 1130081 1130A5R 1130AP5 1130AST  D1130C3W D1130C1B D1130C3C D1130C2P Potentiometer, vertical, Alps RK09K Single, https://tech.alpsalpine.com/prod/e/pdf/potentiometer/rotarypotentiometers/rk09k/rk09k.pdf")
 		(tags "Potentiometer vertical Alps RK09K RK09D Single Snapin")
