File: RC_v2_ESP32/RC_v2_ESP32.kicad_sch (KiCad schematic)
At the start: 13 parts, among them SW3 SW_DIP_x01, SW4 SW_DIP_x01, SW5 SW_DIP_x01, SW6 SW_DIP_x01

Commit message: bearbeitung
Parts:
- removed U2: ~, Amjad_lib:MPU_6050_bord, symbol Amjads_Lib:MPU6050_bord
Other:
- added sheet Power (Power.kicad_sch)
Changed lines of the file:
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@@
-	)
-	(symbol
-		(lib_id "Amjads_Lib:MPU6050_bord")
-		(at 205.74 90.17 0)
-		(unit 1)
-		(exclude_from_sim no)
-		(in_bom yes)
-		(on_board yes)
-		(dnp no)
-		(fields_autoplaced yes)
-		(property "Reference" "U2"
-			(at 208.8041 82.55 0)
-			(effects
-				(font
-					(size 1.27 1.27)
-				)
-				(justify left)
-			)
-		)
-		(property "Value" "~"
-			(at 208.8041 85.09 0)
-			(effects
-				(font
-					(size 1.27 1.27)
-				)
-				(justify left)
-			)
-		)
-		(property "Footprint" "Amjad_lib:MPU_6050_bord"
-			(at 208.8041 86.36 0)
-			(effects
-				(font
-					(size 1.27 1.27)
-				)
-				(justify left)
-			)
-		)
-		(property "Datasheet" ""
-			(at 205.74 90.17 0)
-			(effects
-				(font
-					(size 1.27 1.27)
-				)
-				(hide yes)
-			)
-		)
-		(property "Description" ""
-			(at 205.74 90.17 0)
-			(effects
-				(font
-					(size 1.27 1.27)
-				)
-				(hide yes)
-			)
-		)
-		(pin "4"
-		)
-		(pin "5"
-		)
-		(pin "6"
-		)
-		(pin "3"
-		)
-		(pin "1"
-		)
-		(pin "2"
-		)
-		(pin "7"
-		)
-		(pin "8"
-		)
-		(instances
-			(project ""
-				(path "/f9a7bba8-adff-461f-bcd5-3a30cb8edb3d"
-					(reference "U2")
-					(unit 1)
-				)
-			)
-		)
 	)
 	(symbol
@@
 				)
 			)
+		)
+	)
+	(sheet
+		(at 200.66 86.36)
+		(size 39.37 24.13)
+		(exclude_from_sim no)
+		(in_bom yes)
+		(on_board yes)
+		(dnp no)
+		(fields_autoplaced yes)
+		(stroke
+			(width 0.1524)
+			(type solid)
+		)
+		(fill
+			(color 0 0 0 0.0000)
+		)
+		(property "Sheetname" "Power"
+			(at 200.66 85.6484 0)
+			(effects
+				(font
+					(size 1.27 1.27)
+				)
+				(justify left bottom)
+			)
+		)
+		(property "Sheetfile" "Power.kicad_sch"
+			(at 200.66 111.0746 0)
+			(effects
+				(font
+					(size 1.27 1.27)
+				)
+				(justify left top)
+			)
+		)
+		(instances
+			(project "RC_v2_ESP32"
+				(path "/f9a7bba8-adff-461f-bcd5-3a30cb8edb3d"
+					(page "2")
+				)
+			)
