File: SMT-32_TestBord/SMT-32.kicad_sch (KiCad schematic)
At the start: 33 parts, among them J1 USB_B_Micro, J2 Conn_01x04_Pin, J3 Conn_01x04_Pin, J4 Conn_01x04_Pin, J5 Conn_01x03_Pin, J6 Conn_01x05_Pin, J7 Conn_01x05_Pin, J8 Conn_01x03_Pin, J9 Conn_01x04_Pin, SW1 SW_SPDT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

Commit message: update
design update
Parts:
- removed J5: Conn_01x03_Pin, Connector_PinHeader_2.54mm:PinHeader_1x03_P2.54mm_Vertical, symbol Connector:Conn_01x03_Pin
- added C14: 100n, Capacitor_SMD:C_0402_1005Metric, symbol Device:C
- added J5: Conn_01x02_Socket, Connector_PinSocket_2.54mm:PinSocket_1x02_P2.54mm_Vertical, symbol Connector:Conn_01x02_Socket
Connections:
- net ADC_11: now also J5.1 (Pin_1)
- net ADC_12: now also J5.2 (Pin_2)
- net GND: now also C14.2
- net at J1.6 (Shield): now also C14.1
- no-connect marks 19 -> 17
Other:
- note added: "STM32F103x & USB"
- note removed: "Micro_C & USB"
- moved on the sheet: H1, H2, J1, J8
