File: SMT-32_TestBord/SMT-32.kicad_pcb (KiCad board)
At the start: 4 copper layers, 40 x 33.4 mm, 32 parts, among them J1 USB_B_Micro, J2 Conn_01x04_Pin, J3 Conn_01x04_Pin, J4 Conn_01x04_Pin, J5 Conn_01x03_Pin, J6 Conn_01x05_Pin, J7 Conn_01x05_Pin, J8 Conn_01x03_Pin, SW1 SW_SPDT, U1 STM32F103C8T6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

Commit message: update
design update
Parts:
- added C14: 100n, Capacitor_SMD:C_0402_1005Metric, F.Cu at (112.8, 30.8)
- J5: value Conn_01x03_Pin -> Conn_01x02_Socket; footprint Connector_PinHeader_2.54mm:PinHeader_1x03_P2.54mm_Vertical -> Connector_PinSocket_2.54mm:PinSocket_1x02_P2.54mm_Vertical
- moved H1 0.18 mm to (80.9, 36.2)
- moved H2 0.10 mm to (81.0, 48.1)
Connections:
- J1 pad 6: unconnected-(J1-Shield-Pad6) -> Net-(J1-Shield)
- J5 pad 1: /ADC_12 -> /ADC_11
- J5 pad 2: /ADC_11 -> /ADC_12
Routing:
- net +3.3V: track 79.7 -> 82.6 mm, vias 19 -> 20
- net Net-(J1-Shield): track 0.00 -> 2.82 mm
- net GND: track 71.3 -> 69.2 mm, vias 25 -> 26
Other:
- board text added: "GND"
- board text added: "SPI2"
- board text added: "STM32F103x designed by Amjad Trablsi"
- board text removed: "I2C"
- board text removed: "SPI 2"
