File: Siganl_Generator_ESP32/Siganl_Generator_ESP32.kicad_sch (KiCad schematic)
At the start: 20 parts, among them J1 Conn_01x04_Socket, J2 Conn_01x02_Socket, SW1 SW_Push, SW2 SW_Push, SW3 SW_Push, U2 LM393

Commit message: update
design update
Parts:
- added D3: LED _Red, Diode_SMD:D_1206_3216Metric, symbol Device:LED
- added D4: LED_Green, Diode_SMD:D_1206_3216Metric, symbol Device:LED
- added J4: Conn_01x19_Socket, Connector_PinSocket_2.54mm:PinSocket_1x19_P2.54mm_Vertical, symbol Connector:Conn_01x19_Socket
- added R11, R12: 100, Resistor_SMD:R_1206_3216Metric, symbol Device:R
Connections:
- net 3V3: now also J4.1 (Pin_1), R12.2
- net GND: now also D3.1 (K), D4.1 (K), J4.19 (Pin_19); no longer J2.2 (Pin_2), U2.4 (V-)
- net Signal 1: now also U1.23 (TDX); no longer U1.18 (CMD)
- net Signal 2: now also U1.27 (G19); no longer U1.12 (G14)
- net at U1.10 (G26): now also J4.10 (Pin_10)
- net at U1.11 (G27): now also J4.11 (Pin_11)
- net at U1.13 (G12): now also J4.13 (Pin_13)
- net at U1.15 (G13): now also J4.14 (Pin_14)
- net at U1.16 (SD2): now also J4.15 (Pin_15)
- net at U1.17 (SD3): now also J4.16 (Pin_16)
- net at U1.2 (EN): now also J4.2 (Pin_2)
- net at U1.3 (SP): now also J4.3 (Pin_3)
- net at U1.4 (SN): now also J4.4 (Pin_4)
- net at U1.5 (G34): now also J4.5 (Pin_5)
- net at U1.6 (G35): now also J4.6 (Pin_6)
- net at U1.7 (G32): now also J4.7 (Pin_7)
- net at U1.8 (G33): now also J4.8 (Pin_8)
- net at U1.9 (G25): now also J4.9 (Pin_9)
- net VCC renamed 12 V
- net 12 V: no longer J1.1 (Pin_1), U1.19 (5V)
- new net: D3.2 (A), R11.1
- new net: D4.2 (A), R12.1
- new net: J4.12 (Pin_12), U1.12 (G14)
- new net: J4.17 (Pin_17), U1.18 (CMD)
- new net -12 V: J2.2 (Pin_2), U2.4 (V-)
- new net 5 V: J1.1 (Pin_1), J4.18 (Pin_18), R11.2, U1.19 (5V)
- no-connect marks 0 -> 6
Other:
- added sheet USB-C (untitled.kicad_sch)
- moved on the sheet: D1, D2, J2, R3, R4, R7, R8, R9, SW1, SW2, SW3

Commit message: klein update
Parts:
- added J5: Conn_01x02_Socket, Connector_PinSocket_2.54mm:PinSocket_1x02_P2.54mm_Vertical, symbol Connector:Conn_01x02_Socket
Connections:
- net Siganl 2 Output: now reaches RV4.1, U2.1
- net Siganl 2 Output: now also J5.2 (Pin_2)
- net Signal 1 Output: now reaches RV3.1, U2.7
- net Signal 1 Output: now also J5.1 (Pin_1)
Other:
- moved on the sheet: R2, R6, RV3, RV4, U2A, U2B, U2C

Commit message: update
Parts:
- removed J1: Conn_01x04_Socket, Connector_PinSocket_2.54mm:PinSocket_1x04_P2.54mm_Vertical, symbol Connector:Conn_01x04_Socket
- removed J5: Conn_01x02_Socket, Connector_PinSocket_2.54mm:PinSocket_1x02_P2.54mm_Vertical, symbol Connector:Conn_01x02_Socket
- removed U1: ~, Library_Amjad:ESP_32_socket, symbol Amjad_Lib:ESP32_dev_Socke
- added J1: Conn_01x05_Socket, Connector_PinSocket_2.54mm:PinSocket_1x05_P2.54mm_Vertical, symbol Connector:Conn_01x05_Socket
- added J5, J6: Conn_Coaxial, Connector_Coaxial:SMA_Amphenol_132289_EdgeMount, symbol Connector:Conn_Coaxial
- added U1: ~, Library_Amjad:ESP_32_socket, symbol Amjads_Lib:ESP32_dev_Socke
- R11, R12, R2, R3, R4, R6, R7, R8, R9: footprint Resistor_SMD:R_1206_3216Metric -> Resistor_SMD:R_0603_1608Metric_Pad0.98x0.95mm_HandSolder
Connections:
- net 3V3: now also U1.1 (3V3)
- net 5 V: now also J1.1 (Pin_1), U1.19 (5V)
- net Buttom 1_Siganl_Switch: now also U1.32 (G4)
- net Buttom 2: now also U1.31 (G16)
- net Buttom 3: now also U1.33 (G0)
- net G34 Frquenz: now also U1.34 (G2)
- net G35 DutyCycle: now also U1.35 (G15)
- net GND: now also J1.5 (Pin_5), J5.2 (Ext), J6.2 (Ext), U1.14 (GND), U1.20 (GND), U1.26 (GND)
- net LED_Green: now also U1.25 (G21)
- net Led_Red: now also U1.28 (G18)
- net OLED_SCL: now also J1.2 (Pin_2), U1.22 (G22)
- net OLED_SDA: now also J1.3 (Pin_3), U1.21 (G23)
- net Siganl 2 Output: now also J5.1 (In)
- net Signal 1: now also U1.23 (TDX)
- net Signal 1 Output: now also J6.1 (In)
- net Signal 2: now also U1.27 (G19)
- net at J4.10 (Pin_10): now also U1.10 (G26)
- net at J4.11 (Pin_11): now also U1.11 (G27)
- net at J4.12 (Pin_12): now also U1.12 (G14)
- net at J4.13 (Pin_13): now also U1.13 (G12)
- net at J4.14 (Pin_14): now also U1.15 (G13)
- net at J4.15 (Pin_15): now also U1.16 (SD2)
- net at J4.16 (Pin_16): now also U1.17 (SD3)
- net at J4.17 (Pin_17): now also U1.18 (CMD)
- net at J4.2 (Pin_2): now also U1.2 (EN)
- net at J4.3 (Pin_3): now also U1.3 (SP)
- net at J4.4 (Pin_4): now also U1.4 (SN)
- net at J4.5 (Pin_5): now also U1.5 (G34)
- net at J4.6 (Pin_6): now also U1.6 (G35)
- net at J4.7 (Pin_7): now also U1.7 (G32)
- net at J4.8 (Pin_8): now also U1.8 (G33)
- net at J4.9 (Pin_9): now also U1.9 (G25)
- new net CS: J1.4 (Pin_4)
Other:
- moved on the sheet: R7

Commit message: new design
Parts:
- removed J2: Conn_01x02_Socket, Connector_PinSocket_2.54mm:PinSocket_1x02_P2.54mm_Vertical, symbol Connector:Conn_01x02_Socket
- added R17, R18: 4k7, Resistor_SMD:R_0603_1608Metric_Pad0.98x0.95mm_HandSolder, symbol Device:R
- added TP1, TP3: TestPoint, TestPoint:TestPoint_Pad_D1.0mm, symbol Connector:TestPoint
- added TP5: TestPoint, TestPoint:TestPoint_Pad_D1.5mm, symbol Connector:TestPoint
Connections:
- net -12 V is gone; now on net GND: U2.4 (V-)
- net 3V3: now also R17.1, R18.1
- net 5 V: now also TP3.1
- net Buttom 3: now also U1.12 (G14); no longer U1.33 (G0)
- net G34 Frquenz: now also U1.7 (G32); no longer U1.34 (G2)
- net G35 DutyCycle: now also U1.8 (G33); no longer U1.35 (G15)
- net LED_Green: now also U1.15 (G13); no longer U1.25 (G21)
- net Led_Red: now also U1.9 (G25); no longer U1.28 (G18)
- net OLED_SCL: now also R17.2
- net OLED_SDA: now also U1.25 (G21), R18.2; no longer U1.21 (G23)
- net Siganl 2 Output: now also TP5.1
- net Signal 1: now also U1.5 (G34); no longer U1.23 (TDX)
- net Signal 1 Output: now also TP1.1
- net Signal 2: now also U1.6 (G35); no longer U1.27 (G19)
- net at J4.10 (Pin_10): now also U1.18 (CMD); no longer U1.10 (G26)
- net at J4.11 (Pin_11): no longer U1.11 (G27)
- net at J4.12 (Pin_12): no longer U1.12 (G14)
- net at J4.13 (Pin_13): no longer U1.13 (G12)
- net at J4.14 (Pin_14): no longer U1.15 (G13)
- net at J4.15 (Pin_15): no longer U1.16 (SD2)
- net at J4.16 (Pin_16): no longer U1.17 (SD3)
- net at J4.17 (Pin_17): no longer U1.18 (CMD)
- net at J4.5 (Pin_5): now also U1.10 (G26); no longer U1.5 (G34)
- net at J4.6 (Pin_6): now also U1.11 (G27); no longer U1.6 (G35)
- net at J4.7 (Pin_7): now also U1.13 (G12); no longer U1.7 (G32)
- net at J4.8 (Pin_8): now also U1.16 (SD2); no longer U1.8 (G33)
- net at J4.9 (Pin_9): now also U1.17 (SD3); no longer U1.9 (G25)
- net 12 V renamed 25V
- no-connect marks 6 -> 3
Other:
- note added: "Frequenz"
- note removed: "Frquenz"
- moved on the sheet: J4, U1

Commit message: update
Parts:
- removed U2: LM393, Package_DIP:DIP-8_W7.62mm, symbol Comparator:LM393
- added C8: 100n, Capacitor_SMD:C_0603_1608Metric_Pad1.08x0.95mm_HandSolder, symbol Device:C
- added R19, R20: 50, Resistor_SMD:R_0603_1608Metric_Pad0.98x0.95mm_HandSolder, symbol Device:R
- added U2: NE5532, Package_DIP:DIP-8_W7.62mm, symbol Amplifier_Operational:NE5532
Connections:
- net 25V: now also C8.1, U2.8 (V+)
- net GND: now also C8.2
- net Siganl 2 Output: now also U1.35 (G15), R19.2, U2.1; no longer J5.1 (In), TP5.1
- net Signal 1: now also U2.5 (+)
- net Signal 1 Output: now also R20.2, U2.7; no longer J6.1 (In)
- net Signal 2: now also U2.3 (+)
- net at R6.2, RV4.2: now also U2.2 (-)
- net at R2.2, RV3.2: now also U2.6 (-)
- new net: J6.1 (In), R20.1
- new net: J5.1 (In), R19.1, TP5.1
- new net -25V: U2.4 (V-)
Other:
- moved on the sheet: J4
