File: LED_Array/LED_Driver.kicad_pcb (KiCad board)
At the start: 2 copper layers, 17 parts, among them J1 Conn_01x02_Socket

Commit message: update
Parts:
- moved D15 33.4 mm to (114.2, 51.8), turned to 180 degrees
- moved D3 31.1 mm to (114.3, 67.7), turned to 180 degrees
- moved D7 30.2 mm to (113.3, 82.3), turned to 180 degrees
- moved D11 28.8 mm to (114.4, 37.2), turned to 180 degrees
- moved J1 25.6 mm to (42.5, 76.7)
- moved R2 5.96 mm to (51.5, 83.7)
- moved D5 5.03 mm to (70.3, 81.4)
- moved D6 4.66 mm to (91.7, 82.3)
Routing:
- net GND: track 160.2 -> 48.5 mm
- net Net-(J1-Pin_2): track 65.5 -> 0.79 mm
- net Net-(D6-K): track 23.3 -> 10.0 mm
- net Net-(D10-K): track 19.2 -> 9.75 mm
- net Net-(D14-K): track 16.7 -> 11.1 mm
- net Net-(D5-A): track 9.38 -> 11.2 mm
- net Net-(D5-K): track 11.3 -> 10.3 mm
- removed copper zone on F.Cu, net (none)
Other:
- board outline added: 91.3 x 63.1 mm
