File: boostConverter/boost_converter/boost_converter.kicad_pcb (KiCad board)
At the start: 4 copper layers, 37.5 x 26.8 mm, 22 parts, among them IC1 TPS61175QPWPRQ1, J1 USB_C_Receptacle_PowerOnly_24P

Commit message: update
Parts:
- added J2: Conn_01x06_Socket, Connector_PinHeader_2.00mm:PinHeader_1x06_P2.00mm_Vertical, F.Cu at (160.7, 79.1)
- moved D1 24.2 mm to (131.9, 71.7)
- moved C9 0.45 mm to (155.9, 61.1)
- moved C10 0.24 mm to (157.0, 65.8)
- moved D7 0.18 mm to (150.8, 60.5)
Routing:
- net 25V: track 44.2 -> 76.9 mm, vias 2 -> 4
- net Net-(D5-A_1): track 25.8 -> 38.6 mm, vias 0 -> 2
- net -25V: track 5.49 -> 14.8 mm
- net GND: track 28.4 -> 34.0 mm, vias 21 -> 24
- net unconnected-(J1-SHIELD-PadS1): track 0.00 -> 5.21 mm, vias 0 -> 4
- net 5 V: track 55.7 -> 52.9 mm, vias 3 -> 4
- added copper zone on F.Cu, net 25V
- added copper zone on F.Cu, net 5 V
Other:
- board size 37.5 x 26.8 mm -> 40.5 x 26.7 mm
- board text added: "+ +"
- board text added: "- -"
- board text added: "GND GND"
